File: Eagle/apollo18.sch (EAGLE design)
At the start: 29 parts, among them IC1 L298, IC2 7808T, IC3 7808T, IC4 7805T, IC5 7805T, IC6 7805T

Commit message: Update Eagle CAD PCB files
Parts:
- removed IC3: 7808T, linear:7808T
- removed IC5: 7805T, linear:7805T
- added D2, D3, D4, D5, D6, D7, D8, D9: 1N4004, diode:1N4004
- added J5, J9: (no value), con-amp:MTA10-100
- C4: device rcl:C-US025-050X050 -> rcl:C-US025-025X050
Connections:
- net +12V: now also D3.C, D4.C, D5.C, D6.C
- net +5V: no longer IC5.VO
- net AN1: now also U$1.P1.3; no longer U$1.P1.0
- net AN2: now also U$1.P1.0; no longer U$1.P1.3
- net GND: now also D2.A, D7.A, D8.A, D9.A; no longer IC3.GND, IC5.GND
- net N$2: now also D2.C, D3.A
- net N$3: now also D4.A, D7.C
- net N$4: now also D5.A, D8.C
- net N$5: now also D6.A, D9.C
- net N$6: no longer IC3.VI
- net N$8: no longer IC3.VO, IC5.VI
Other:
- moved on the sheet: J1, J2, J3, J4, J6, J8, R1, R2
